File: Projects/Differential/Diff2rev4/Diff2rev4.kicad_pcb (KiCad board)
At the start: 2 copper layers, 53 x 40.9 mm, 42 parts, among them J1 AVR-ISP-6, J3 12401598E4_2A, U1 ATmega32U4-M, U2 DRV8904QPWPRQ1, U3 AP7363-33D-13, Y1 C5S-24.000-20-3030-X-R

Commit message: chore: clean kicad schematics
Changed lines of the file:
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@@
 		(min_thickness 0.25)
 		(filled_areas_thickness no)
-		(fill yes
+		(fill
 			(thermal_gap 0.5)
 			(thermal_bridge_width 0.5)
@@
 		(polygon
 			(pts
-				(xy 210.9 107.32) (xy 213.614 75.599) (xy 146.812 75.853) (xy 145.796 126.399) (xy 217.678 126.907)
+				(xy 216.5 104) (xy 220 68) (xy 141.5 73.5) (xy 138.5 136.5) (xy 217.678 126.907)
 			)
 		)
